Commit message: Prepare portable FR5 line-scanner deployment

File: ros2_fr5/src/fairino_description/urdf/fairino5_v6.urdf (robot description, URDF)
Before this commit: robot fairino5_v6_robot, 7 links, 6 joints
Links:
- added link fairino_flange_model
- added link hik_450_camera_optical_frame
- added link hik_camera_optical_frame
- added link scanner_650_body; collision box size=0.18 0.16 0.20; visual box size=0.18 0.16 0.20
- added link scanner_650_scan_tcp
Joints:
- added joint fairino_flange_model_to_hik_450_camera_optical: type fixed, parent fairino_flange_model, child hik_450_camera_optical_frame, origin xyz=0.0658967727891 -0.00975216317425 0.126228380771 rpy=0.508947894454 -0.004857842133 3.134367571689
- added joint fairino_flange_model_to_hik_camera_optical: type fixed, parent fairino_flange_model, child hik_camera_optical_frame, origin xyz=-0.0608482323161 -0.000382077753729 0.142143365159 rpy=0.522159631925 0.006209883087 3.140900573284
- added joint fairino_flange_model_to_scanner_650_body: type fixed, parent fairino_flange_model, child scanner_650_body, origin xyz=0 0 0 rpy=0 0 0
- added joint hik_camera_optical_to_scanner_650_scan_tcp: type fixed, parent hik_camera_optical_frame, child scanner_650_scan_tcp, origin xyz=0 0.0466476147 0.55 rpy=0 0 1.57079632679
- added joint wrist3_to_fairino_flange_model: type fixed, parent wrist3_link, child fairino_flange_model, origin xyz=0 0 0.1 rpy=0 0 0
